File: PCDB_project/Comm.sch (KiCad schematic (older format))
At the start: 9 parts, among them J6 Comm, M2 BSS84, U5 MAX3486

Commit message: BOM añadido y comprobado las footprints, en principio estan bien. falta ocnfirmar con el profesor y medir el boton que parece que no estoy seguro si están bien hechos los pines
Parts:
- J6: footprint (none) -> PCDB_project:IO3
Changed lines of the file:
@@
 F 0 "J6" H 7980 2442 50  0000 L CNN
 F 1 "Comm" H 7980 2351 50  0000 L CNN
-F 2 "" H 7900 2400 50  0001 C CNN
+F 2 "PCDB_project:IO3" H 7900 2400 50  0001 C CNN
 F 3 "~" H 7900 2400 50  0001 C CNN
 F 4 "22-05-7025" H 7900 2400 50  0001 C CNN "Name"
