File: PCDB_project/OneWire.sch (KiCad schematic (older format))
At the start: 5 parts, among them J2 22-05-7025, M1 BSS84, U4 DS1822-PAR

Commit message: BOM añadido y comprobado las footprints, en principio estan bien. falta ocnfirmar con el profesor y medir el boton que parece que no estoy seguro si están bien hechos los pines
Parts:
- J2: footprint (none) -> PCDB_project:IO2
Changed lines of the file:
@@
 F 0 "J2" H 5830 1742 50  0000 L CNN
 F 1 "22-05-7025" H 5830 1651 50  0000 L CNN
-F 2 "" H 5750 1750 50  0001 C CNN
+F 2 "PCDB_project:IO2" H 5750 1750 50  0001 C CNN
 F 3 "~" H 5750 1750 50  0001 C CNN
 F 4 "22-05-7025" H 5750 1750 50  0001 C CNN "Name"
