File: PCDB_project/mcu.sch (KiCad schematic (older format))
At the start: 15 parts, among them SW1 Reset, U3 STM32F103CBT6, X1 8MHz

Commit message: BOM añadido y comprobado las footprints, en principio estan bien. falta ocnfirmar con el profesor y medir el boton que parece que no estoy seguro si están bien hechos los pines
Parts:
- SW1: footprint (none) -> PCDB_project:B3F-4000
Changed lines of the file:
@@
 F 0 "SW1" V 1246 2352 50  0000 R CNN
 F 1 "Reset" V 1155 2352 50  0000 R CNN
-F 2 "" H 1200 2600 50  0001 C CNN
+F 2 "PCDB_project:B3F-4000" H 1200 2600 50  0001 C CNN
 F 3 "~" H 1200 2600 50  0001 C CNN
 F 4 "B3F-400" H 1200 2400 50  0001 C CNN "Name"
