File: PCDB_project/supply.sch (KiCad schematic (older format))
At the start: 13 parts, among them J1 Power, U1 TSR_1-2450, U2 UA78M33

Commit message: BOM añadido y comprobado las footprints, en principio estan bien. falta ocnfirmar con el profesor y medir el boton que parece que no estoy seguro si están bien hechos los pines
Parts:
- J1: footprint (none) -> PCDB_project:Power
- L1: footprint (none) -> PCDB_project:tck141
Connections:
- net pwr1: now reaches F1.2, J1.2 (Pin_2)
- net pwr2: now reaches C1.1, F1.1, L1.1
- net pwr3: now reaches C2.1, L1.2, U1.1 (Vin)
- net pwr5: now reaches C3.1, D1.1 (K), D2.1 (K), U2.1 (IN)
- net pwr4: now reaches D1.2 (A), U1.3 (Vout)
Changed lines of the file:
@@
 F 0 "J1" H 1768 1975 50  0000 C CNN
 F 1 "Power" H 1768 2066 50  0000 C CNN
-F 2 "" H 1850 2300 50  0001 C CNN
+F 2 "PCDB_project:Power" H 1850 2300 50  0001 C CNN
 F 3 "~" H 1850 2300 50  0001 C CNN
 F 4 "20.101M/2" H 1768 1975 50  0001 C CNN "Name"
@@
 F 0 "L1" V 3831 2200 50  0000 C CNN
 F 1 "5.6uH" V 3740 2200 50  0000 C CNN
-F 2 "" H 3550 2200 50  0001 C CNN
+F 2 "PCDB_project:tck141" H 3550 2200 50  0001 C CNN
 F 3 "~" H 3550 2200 50  0001 C CNN
 F 4 "tck141" V 3649 2200 50  0000 C CNN "Name"
@@
 	1    0    0    -1
 $EndComp
+Text Label 2250 2200 0    50   ~ 0
+pwr1
+Text Label 3050 2200 0    50   ~ 0
+pwr2
+Text Label 3750 2200 0    50   ~ 0
+pwr3
+Text Label 5000 2200 0    50   ~ 0
+pwr4
+Text Label 5700 2200 0    50   ~ 0
+pwr5
 $EndSCHEMATC
