File: PCDB_project/usb-debug.sch (KiCad schematic (older format))
At the start: 3 parts, among them J7 USB_B_Mini, J8 Debug

Commit message: BOM añadido y comprobado las footprints, en principio estan bien. falta ocnfirmar con el profesor y medir el boton que parece que no estoy seguro si están bien hechos los pines
Parts:
- J8: footprint (none) -> PCDB_project:Debug
Changed lines of the file:
@@
 F 0 "J8" H 5680 1992 50  0000 L CNN
 F 1 "Debug" H 5680 1901 50  0000 L CNN
-F 2 "" H 5600 2000 50  0001 C CNN
+F 2 "PCDB_project:Debug" H 5600 2000 50  0001 C CNN
 F 3 "~" H 5600 2000 50  0001 C CNN
 F 4 "T821106A1S100CEU" H 5600 2000 50  0001 C CNN "Name"

Commit message: Placement acabado pero hay algunas dudas que resolver con el profe
Connections:
- net GND: now also J7.5 (GND), J7.6 (Shield), R2.2
Changed lines of the file:
@@
 Connection ~ 3400 2750
 Wire Wire Line
-	3400 2750 4050 2750
+	3400 2750 3800 2750
 Wire Wire Line
 	5300 2450 5300 2300
@@
 Wire Wire Line
 	5250 1800 5400 1800
+Wire Wire Line
+	3800 2750 3800 2850
+Connection ~ 3800 2750
+Wire Wire Line
+	3800 2750 4050 2750
 $EndSCHEMATC
