File: PCDB_project/PCDB_project.kicad_pcb (KiCad board)
At the start: 4 copper layers, 100 x 80 mm, 66 parts, among them J1 Power, J2 22-05-7025, J3 22-05-7025, J4 22-05-7025, J5 22-05-7025, J6 Comm, J7 USB_B_Mini, J8 Debug, M1 BSS84, M2 BSS84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

Commit message: Version final PCDB
Parts:
- moved C12 48.0 mm to (60.1, 44.1), turned to 90 degrees
- moved R3 44.3 mm to (58.0, 44.0)
Routing:
- net Net-(U3-Pad17): track 37.9 -> 0.00 mm
- net ALARM_C: track 59.5 -> 70.4 mm
- net NRST: track 178.9 -> 172.6 mm
- net +3V3: track 90.7 -> 95.1 mm, vias 14 -> 15
- net FAN2_C: track 71.7 -> 67.4 mm
- net Net-(LD2-Pad1): track 152.8 -> 150.3 mm
