File: PCDB_project_2_layer/PCDB_project.kicad_pcb (KiCad board)
At the start: 2 copper layers, 100 x 80 mm, 66 parts, among them J1 Power, J2 22-05-7025, J3 22-05-7025, J4 22-05-7025, J5 22-05-7025, J6 Comm, J7 USB_B_Mini, J8 Debug, M1 BSS84, M2 BSS84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

Commit message: Version final PCDB
Parts:
- moved R3 47.3 mm to (62.7, 46.7)
- moved C12 46.0 mm to (57.8, 44.0), turned to 90 degrees
- moved C5 1.25 mm to (41.7, 56.9), turned to 180 degrees
Routing:
- net NRST: track 63.6 -> 97.0 mm, vias 1 -> 2
- net FAN1_C: track 44.0 -> 57.7 mm
- net ALARM_C: track 59.5 -> 68.2 mm
- net FAN2_C: track 71.7 -> 67.3 mm, vias 0 -> 2
- net SWCLK: track 26.2 -> 23.6 mm
- net Net-(LD2-Pad1): track 152.8 -> 150.2 mm
- net +3V3: track 32.9 -> 30.7 mm, vias 5 -> 2
- net SWDIO: track 26.2 -> 24.0 mm
- net Net-(LD6-Pad1): track 40.1 -> 41.2 mm
- net Net-(J4-Pad1): track 38.9 -> 39.7 mm
