File: PCDB_project_miled/PCDB_project.kicad_pcb (KiCad board)
At the start: 2 copper layers, 100 x 80 mm, 120 parts, among them J1 Power, J2 22-05-7025, J3 22-05-7025, J4 22-05-7025, J5 22-05-7025, J6 Comm, J7 USB_B_Mini, J8 Debug, M1 BSS84, M2 BSS84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

Commit message: Version final PCDB
Parts:
- moved REF** 11.5 mm to (64.0, 45.7)
Routing:
- net NRST: track 70.5 -> 102.6 mm
